File: FR4 Case/fr4/fr4.kicad_pcb (KiCad board)
At the start: 2 copper layers, 304.4 x 131.1 mm, 0 parts

Commit message: Big update of everything exept the PCB
Routing:
- net (no net): track 0.00 -> 1.12 mm
Other:
- board size 304.4 x 131.1 mm -> 325.2 x 131.1 mm
